Commit message: feat(robotiq_description): add hardware support for the Hand-E C10
- hand_e_c10.ros2_control.xacro and its wiring in the C10 macro: finger 1 is the
  one commanded joint, the other two follow it through <mimic>; the real driver,
  the mock hardware and the topic-based simulation use the same arguments as the
  other models, and the driver takes the joint's speed and force limits
- robotiq_control.launch.py: hand_e_c10 in the joint, goal tolerance and stall
  velocity tables
- robotiq_driver: the hand_e_c10 gripper_profile, from the SDK's kHandEC10
- tests: the C10 joins the parametrized model, profile and Humble-launch tests;
  the test that said it had no ros2_control block now checks the block
- README

Needs the SDK's kHandEC10 (robotiq/grippers#80).

File: grippers/robotiq_description/urdf/robotiq_hand_e_c10_macro.urdf.xacro (robot description, xacro)
@@ -1,8 +1,7 @@
 <?xml version="1.0"?>
 <!-- Robotiq Hand-E C10: three concentric fingers, 120 degrees apart, that slide radially toward the gripper axis.
-     A description without control support: links, joints, meshes and inertia, for visualization, planning and
-     URDF-importing simulators. There is no <ros2_control> block, so there is no driver, mock or simulated control
-     yet (hardware support is tracked in #150); the hardware arguments below are accepted, so the shared
-     robotiq_gripper.urdf.xacro can instantiate it with gripper_model:=hand_e_c10, and ignored.
+     Hardware support: the <ros2_control> block (hand_e_c10.ros2_control.xacro) drives hande_c10_finger_1_joint, the
+     other two fingers follow it through <mimic>. The real driver, the mock hardware and the topic-based simulation
+     are selected by the same arguments as for the other models.
      Frame: origin on the gripper axis at the mounting flange (the back face of the housing), +Z toward the
      fingertips, finger 1 along +X, finger 2 at +120 degrees and finger 3 at +240 degrees about Z.
@@ -33,5 +32,5 @@
         use_fake_hardware:=false
         mock_sensor_commands:=false
-        include_ros2_control:=false
+        include_ros2_control:=true
         com_port:=/dev/ttyUSB0
         baudrate:=115200
@@ -39,7 +38,12 @@
         gripper_force_multiplier:=0.5
         tcp_z_offset:=0.15477">
-        <xacro:if value="${include_ros2_control}">
-            ${xacro.warning('the Hand-E C10 description has no ros2_control block yet; include_ros2_control is ignored')}
+        <!-- PickNik's names for the topic-based path, released in 1.1.0 and
+             deprecated since 1.2.0; an explicit new-style argument wins over both. -->
+        <xacro:if value="${sim_isaac or isaac_joint_commands != '' or isaac_joint_states != ''}">
+            ${xacro.warning('sim_isaac, isaac_joint_commands and isaac_joint_states are deprecated since 1.2.0 and removed in the next major release; use sim_topic_based, sim_joint_commands_topic and sim_joint_states_topic')}
         </xacro:if>
+        <xacro:property name="topic_based" value="${sim_topic_based or sim_isaac}"/>
+        <xacro:property name="commands_topic" value="${isaac_joint_commands or ('/isaac_joint_commands' if sim_isaac else sim_joint_commands_topic)}"/>
+        <xacro:property name="states_topic" value="${isaac_joint_states or ('/isaac_joint_states' if sim_isaac else sim_joint_states_topic)}"/>
         <!-- One finger's radial travel, 0 open to fully closed (CAD: the fingers go from 51.3 mm to 32.1 mm from the
              axis, so the diameter between the fingertips changes by 38.5 mm; the datasheet quotes 40 mm). -->
@@ -49,4 +53,23 @@
         <!-- Datasheet maximum grip force, per finger. -->
         <xacro:property name="finger_effort" value="175.0"/>
+        <xacro:include filename="$(find robotiq_description)/urdf/hand_e_c10.ros2_control.xacro" />
+        <xacro:if value="${include_ros2_control}">
+            <!-- The driver's full speed and force are the finger joint's limits, and it closes at one finger's travel. -->
+            <xacro:robotiq_gripper_ros2_control
+                name="${name}" prefix="${prefix}"
+                sim_gazebo="${sim_gazebo}"
+                sim_topic_based="${topic_based}"
+                sim_joint_commands_topic="${commands_topic}"
+                sim_joint_states_topic="${states_topic}"
+                use_fake_hardware="${use_fake_hardware}"
+                mock_sensor_commands="${mock_sensor_commands}"
+                com_port="${com_port}"
+                baudrate="${baudrate}"
+                gripper_speed_multiplier="${gripper_speed_multiplier}"
+                gripper_force_multiplier="${gripper_force_multiplier}"
+                gripper_max_speed="${finger_speed}"
+                gripper_max_force="${finger_effort}"
+                gripper_closed_position="${travel}"/>
+        </xacro:if>
         <link name="${prefix}hand_e_c10_base_link">
             <inertial>
