Commit message: fix(robotiq_description): address review of the Hand-E C10 hardware support
- wrap the profile error in hardware_parameters.cpp (ament_cpplint, Format)
- the C10 macro takes gripper_max_speed, gripper_max_force and
  gripper_closed_position like the other models, with empty defaults that fall
  back to its properties
- declare the C10's followers for Gazebo only, so the topic-based simulation
  sees one joint (#118)
- split the speed and force checks into separate tests, and test the macro's
  arguments and the Gazebo followers
- fix the stall-velocity comment (the slowest C10 finger speed is 0.007 m/s)
  and re-wrap the goal-tolerance comment
- drop the not-measured caveats: the endpoints and the speed reading were
  measured on a C10

File: grippers/robotiq_description/urdf/hand_e_c10.ros2_control.xacro (robot description, xacro)
@@ -56,5 +56,8 @@
                 </xacro:unless>
             </joint>
-            <xacro:if value="${sim_topic_based or sim_gazebo}">
+            <!-- The followers are declared for Gazebo only, as proposed for #118: under sim_topic_based a declared mimic joint
+                 makes the simulator's command name more joints than it gives positions for. /joint_states carries them
+                 through <mimic> in robot_state_publisher. -->
+            <xacro:if value="${sim_gazebo}">
                 <xacro:robotiq_sim_mimic_joint name="${prefix}hande_c10_finger_2_joint" sim_gazebo="${sim_gazebo}"/>
                 <xacro:robotiq_sim_mimic_joint name="${prefix}hande_c10_finger_3_joint" sim_gazebo="${sim_gazebo}"/>

File: grippers/robotiq_description/urdf/robotiq_hand_e_c10_macro.urdf.xacro (robot description, xacro)
@@ -37,4 +37,7 @@
         gripper_speed_multiplier:=1.0
         gripper_force_multiplier:=0.5
+        gripper_max_speed:=''
+        gripper_max_force:=''
+        gripper_closed_position:=''
         tcp_z_offset:=0.15477">
         <!-- PickNik's names for the topic-based path, released in 1.1.0 and
@@ -55,5 +58,7 @@
         <xacro:include filename="$(find robotiq_description)/urdf/hand_e_c10.ros2_control.xacro" />
         <xacro:if value="${include_ros2_control}">
-            <!-- The driver's full speed and force are the finger joint's limits, and it closes at one finger's travel. -->
+            <!-- The other models take gripper_max_speed, gripper_max_force and gripper_closed_position with defaults of their own;
+                 here an empty default falls back to the properties below, so each value still has one home: the driver's full
+                 speed and force are the finger joint's limits, and it closes at one finger's travel. -->
             <xacro:robotiq_gripper_ros2_control
                 name="${name}" prefix="${prefix}"
@@ -68,7 +73,7 @@
                 gripper_speed_multiplier="${gripper_speed_multiplier}"
                 gripper_force_multiplier="${gripper_force_multiplier}"
-                gripper_max_speed="${finger_speed}"
-                gripper_max_force="${finger_effort}"
-                gripper_closed_position="${travel}"/>
+                gripper_max_speed="${gripper_max_speed or finger_speed}"
+                gripper_max_force="${gripper_max_force or finger_effort}"
+                gripper_closed_position="${gripper_closed_position or travel}"/>
         </xacro:if>
         <link name="${prefix}hand_e_c10_base_link">
